File: pcb/pendant.brd (EAGLE design)
At the start: 24 x 100 mm, 76 parts, among them CON1 USB_MICROSMT+THRUHULE, Q2 16MHz, SW2 BUTTON_2, T1 SSM3J328R,LF, T2 SSM3J328R,LF, U2 MK20D--VFM5, U3 74LVC1G17DCK, U4 74LVC1G17DCK

Commit message: Update reference designators
Parts:
- removed C13: 100nF, adafruit:C0402
- removed U$6: MMA8653FC, teensy_adapter:VFDFN-10
- added C4: 100nF, adafruit:C0402
- added U1: MK20D--VFM5, blinkinlabs:QFN32_5X5_LONGLEADS
- U2: value MK20D--VFM5 -> MMA8653FC; device blinkinlabs:QFN32_5X5_LONGLEADS -> teensy_adapter:VFDFN-10
- moved C5 11.0 mm to (8.25, 12.8), turned to 180 degrees
- moved U2 7.57 mm to (12.0, 23.0), turned to 180 degrees
- renumbered C11 to C6, C12 to C10, C14 to C8, C15 to C7, C17 to C9, U$1 to CON2, U$2 to SW1, U4 to U5
Connections:
- net +5V: now also U1.6; no longer U2.6
- net 3.3V: now also C4.1, U1.1, U1.11, U1.5, U1.7, U2.P$1, U2.P$8; no longer C13.1, U$6.P$1, U$6.P$8, U2.1, U2.11, U2.5, U2.7
- net ACC_INT1: now also U1.24, U2.P$3; no longer U$6.P$3, U2.24
- net GND: now also C4.2, U1.2, U1.8, U1.PAD@1, U1.PAD@11, U1.PAD@4, U1.PAD@9, U2.P$6, U2.P$7, U2.P$9; no longer C13.2, U$6.P$6, U$6.P$7, U$6.P$9, U2.2, U2.8, U2.PAD@1, U2.PAD@11, U2.PAD@4, U2.PAD@9
- net I2C0_SCL: now also U1.20, U2.P$2; no longer U$6.P$2, U2.20
- net I2C0_SDA: now also U1.21, U2.P$10; no longer U$6.P$10, U2.21
- net LED_CLOCK: now also U1.26; no longer U2.26
- net LED_DATA: now also U1.27; no longer U2.27
- net LED_OE: now also U1.16; no longer U2.16
- net LED_S0: now also U1.29; no longer U2.29
- net LED_S1: now also U1.30; no longer U2.30
- net LED_STROBE: now also U1.31; no longer U2.31
- net N$13: now also U1.18; no longer U2.18
- net N$15: now also U1.4; no longer U2.4
- net N$17: now also U1.3; no longer U2.3
- net N$4: now also U2.P$4; no longer U$6.P$4
- net N$8: now also U1.17; no longer U2.17
- net RESET: now also U1.19; no longer U2.19
- net RX: now also U1.13; no longer U2.13
- net TCLK: now also U1.12; no longer U2.12
- net TMS: now also U1.15; no longer U2.15
- net TX: now also U1.14; no longer U2.14
