File: testjig/pcb/controller testjig.brd (EAGLE design)
At the start: 80 x 75 mm, 50 parts, among them IC1 AD8041R, J1 POWER_JACKPTH, SW2 BUTTON_2

Commit message: Update board
Changed lines of the file:
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@@
 <attribute name="VALUE" x="17.214" y="54.889" size="1.27" layer="27" rot="SR270"/>
 </element>
-<element name="JP2" library="SparkFun-Connectors" package="USB-A-H" value="USB-A-H" x="9.5" y="46.5">
+<element name="JP2" library="SparkFun-Connectors" package="USB-A-H" value="USB-A-H" x="9.5" y="46.5" smashed="yes">
 <attribute name="PROD_ID" value="CONN-08367" x="9.5" y="46.5" size="1.778" layer="27" display="off"/>
 </element>

Commit message: Bringing up the test rig
Connections:
- net TARGET_001_MEAS renamed TARGET_VBAT_MEAS
Changed lines of the file:
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@@
 <via x="33" y="64" extent="1-16" drill="0.35"/>
 </signal>
-<signal name="TARGET_001_MEAS">
+<signal name="TARGET_VBAT_MEAS">
 <contactref element="U$1" pad="14/A0"/>
 <contactref element="R9" pad="1"/>

Commit message: Add S0, S1 tests, begin I2C work for accelerometer
Connections:
- net TARGET_002_MEAS renamed TARGET_S0_MEAS
- net TARGET_003_MEAS renamed TARGET_S1_MEAS
Changed lines of the file:
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@@
 <via x="29" y="60" extent="1-16" drill="0.35"/>
 </signal>
-<signal name="TARGET_003_MEAS">
+<signal name="TARGET_S1_MEAS">
 <contactref element="U$1" pad="16/A2"/>
 <contactref element="R11" pad="1"/>
@@
 <via x="31" y="62" extent="1-16" drill="0.35"/>
 </signal>
-<signal name="TARGET_002_MEAS">
+<signal name="TARGET_S0_MEAS">
 <contactref element="U$1" pad="15/A1"/>
 <contactref element="R10" pad="1"/>

Commit message: Fix target poweroff routine, add nonworking LED test
Connections:
- new net POWER_RESET: U$1.9
Changed lines of the file:
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@@
 <wire x1="16.5" y1="58.85" x2="16.5" y2="60.65" width="0.254" layer="1"/>
+</signal>
+<signal name="POWER_RESET">
+<contactref element="U$1" pad="9"/>
 </signal>
 </signals>
